File: hw-keeb-pcb.kicad_pcb (KiCad board)
At the start: 2 copper layers, 73.8 x 38.1 mm, 24 parts, among them SW1 SW_Push, U1 ATmega32U4-AU, Y1 16MHz

Commit message: Base matrix schematic added.
Other:
- net class Default removed

Commit message: Gitignore update.
Parts:
- removed C1, C2, C3, C6: 0.1uF, Capacitor_SMD:C_0805_2012Metric
- removed C4, C5: 22pF, Capacitor_SMD:C_0805_2012Metric
- removed C7: 1uF, Capacitor_SMD:C_0805_2012Metric
- removed D1, D2, D3, D4: D_Small, Diode_SMD:D_SOD-123
- removed F1: 500mA, Fuse:Fuse_1206_3216Metric
- removed MX1, MX2, MX3, MX4: MX-1U, MX_Alps_Hybrid:MX-1U
- removed R1, R2: 22, Resistor_SMD:R_0805_2012Metric
- removed R3: 10K, Resistor_SMD:R_0805_2012Metric
- removed R4: 10k, Resistor_SMD:R_0805_2012Metric
- removed SW1: SW_Push, random-keyboard-parts:SKQG-1155865
- removed U1: ATmega32U4-AU, Package_QFP:PQFP-44_10x10mm_P0.8mm
- removed USB1: Molex-0548190589, random-keyboard-parts:Molex-0548190589
- removed Y1: 16MHz, Crystal:Crystal_SMD_3225-4Pin_3.2x2.5mm
Other:
- board outline removed
