File: hw-keeb-pcb.kicad_sch (KiCad schematic)
At the start: 178 parts

Commit message: Schematic finish touches.
Parts:
- C1, C2: renamed from C?; value C_Small -> 22pF
- C3: renamed from C?; value C_Small -> 1uF
- C4: renamed from C?; value C_Small -> 10uF
- C5, C6, C7: renamed from C?; value C_Small -> 0.1uF
- R1: renamed from R?; value R_Small -> 10K
- R4: renamed from R?; value R_Small -> 1k
- SW1: renamed from SW?; value SW_Push -> 5.2x5.2mm
- U1: renamed from U?; value ATmega32U4-AU-MCU_Microchip_ATmega -> ATmega32U4-AU
- Y1: renamed from Y?; value Crystal_GND24_Small-Device -> 16Mhz
- gave numbers to parts that had none: 166
Connections:
- net COL0: now also U1.36 (PF7)
- net COL1: now also U1.37 (PF6)
- net COL10: now also U1.26 (PD6)
- net COL11: now also U1.25 (PD4)
- net COL12: now also U1.22 (PD5)
- net COL13: now also U1.21 (PD3)
- net COL14: now also U1.20 (PD2)
- net COL2: now also U1.38 (PF5)
- net COL3: now also U1.32 (PC7)
- net COL4: now also U1.31 (PC6)
- net COL5: now also U1.12 (PB7)
- net COL6: now also U1.30 (PB6)
- net COL7: now also U1.29 (PB5)
- net COL8: now also U1.28 (PB4)
- net COL9: now also U1.27 (PD7)
- net RGBLED: now also U1.19 (PD1); no longer U1.20 (PD2)
- net ROW0: now also U1.9 (PB1)
- net ROW1: now also U1.10 (PB2)
- net ROW2: now also U1.11 (PB3)
- net ROW3: now also U1.41 (PF0)
- net ROW4: now also U1.40 (PF1)
- net ROW5: now also U1.39 (PF4)
